File: hive_access_pcb.kicad_pcb (KiCad board)
At the start: 2 copper layers, 43 parts, among them J1 Door Reader, J2 Snub Enable, J3 Relay Mode Select, J4 Relay Voltage Select, J5 Power In, J6 Exit Sensor, K1 SANYOU_SRD_Form_C, P1 Door Latch Solenoid Out, P2 External Reset, P3 Door Closed Sensor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

Commit message: Basic layout.
Parts:
- moved R11 116.9 mm to (148.6, 118.1), turned to 180 degrees
- moved R12 113.7 mm to (148.6, 124.5), turned to 180 degrees
- moved U3 113.6 mm to (150.0, 154.9)
- moved R10 113.1 mm to (153.0, 118.1)
- moved R13 112.5 mm to (152.4, 124.5)
- moved J6 97.8 mm to (170.8, 135.3), turned to 90 degrees
- moved Q6 93.4 mm to (158.8, 132.1)
- moved C5 93.0 mm to (115.0, 116.8)
- moved C2 89.0 mm to (120.1, 164.5)
- moved R9 88.7 mm to (137.2, 135.9)
- moved U2 85.6 mm to (151.8, 132.1)
- moved P1 84.2 mm to (99.1, 121.3), turned to 270 degrees
- moved Q1 83.2 mm to (123.2, 101.6)
- moved Q5 83.2 mm to (168.9, 119.4)
- moved Q4 81.5 mm to (130.2, 101.6)
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Other:
- net class 3.3V added: clearance 0.2032, trace_width 0.762, via_dia 1.016, via_drill 0.508
- net class Default: clearance 0.2 -> 0.2032; trace_width 0.25 -> 0.254; via_dia 0.6 -> 0.762; via_drill 0.4 -> 0.4064
- net class Power added: clearance 0.2032, trace_width 1.524, via_dia 2.032, via_drill 1.397
- rule trace_clearance: 0.2 -> 0.2032

Commit message: First draft of actual PCB.
Parts:
- added REF**: 1pin, Connectors:1pin, F.Cu at (172.7, 82.5)
- added REF**: 1pin, Connectors:1pin, F.Cu at (172.7, 171.4)
- added REF**: 1pin, Connectors:1pin, F.Cu at (96.5, 171.4)
- added REF**: 1pin, Connectors:1pin, F.Cu at (96.5, 82.5)
- moved P2 38.7 mm to (132.1, 170.2), turned to 0 degrees
- moved R1 20.3 mm to (153.0, 90.8), turned to 0 degrees
- moved R13 10.2 mm to (162.6, 124.5), turned to 180 degrees
- moved C1 4.45 mm to (101.6, 165.1)
- moved J5 3.70 mm to (109.2, 170.2)
- moved J3 2.54 mm to (95.9, 91.4)
Routing:
- net GND: track 0.00 -> 464.3 mm
- net +12V: track 0.00 -> 243.5 mm
- net +5V: track 0.00 -> 217.4 mm
- net +3V3: track 0.00 -> 214.9 mm
- net /DOOR_OPEN: track 0.00 -> 101.5 mm
- net /WEMOS_D0: track 0.00 -> 85.3 mm
- net /WEMOS_D1: track 0.00 -> 77.6 mm
- net /WEMOS_ECHO: track 0.00 -> 71.7 mm
- net /RELAY_POWER: track 0.00 -> 66.4 mm
- net /WIEGAND_BEEP: track 0.00 -> 63.3 mm, vias 0 -> 1
- net /WEMOS_TRIG: track 0.00 -> 60.6 mm
- net /WIEGAND_LIGHT: track 0.00 -> 60.5 mm, vias 0 -> 1
- net /ONE_WIRE: track 0.00 -> 56.3 mm
- net /RELAY_CONN: track 0.00 -> 55.6 mm
- net /~RST: track 0.00 -> 48.6 mm
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Other:
- board outline added: 82.6 x 95.2 mm
- board text added: "+12"
- board text added: "12"
- board text added: "5"
- board text added: "Jumper inner two to have the relay short P1. Jumper both outers to apply +12V to P1."
- board text added: "Relay Mode Select"

Commit message: Fix issues.
Parts:
- moved J2 14.1 mm to (99.7, 107.3)
- moved D3 10.2 mm to (109.2, 106.0)
- moved R10 9.53 mm to (162.6, 118.1), turned to 180 degrees
- moved R5 9.53 mm to (153.0, 86.4), turned to 0 degrees
- moved D1 3.18 mm to (101.0, 114.9)
- moved R7 0.64 mm to (146.1, 95.2)
Connections:
- K1 pad 3: Net-(K1-Pad3) -> /RELAY_CONTACT
- K1 pad 4: /RELAY_CONTACT -> Net-(K1-Pad4)
- R10 pad 1: +3V3 -> /WEMOS_TRIG
- R10 pad 2: /WEMOS_TRIG -> +3V3
- R5 pad 1: +3V3 -> /WEMOS_D0
- R5 pad 2: /WEMOS_D0 -> +3V3
- U3 pad 10: Net-(U3-Pad10) -> +3V3
- U4 pad 12: Net-(U4-Pad12) -> /WEMOS_ECHO
- U4 pad 15: /WEMOS_ECHO -> Net-(U4-Pad15)
Routing:
- net /RELAY_CONN: track 55.6 -> 33.7 mm
- net /WIEGAND_D1: track 48.3 -> 61.5 mm
- net /WEMOS_ECHO: track 71.7 -> 60.7 mm
- net /WIEGAND_BEEP: track 63.3 -> 54.5 mm
- net /WIEGAND_LIGHT: track 60.5 -> 52.4 mm
- net +3V3: track 214.9 -> 220.8 mm, vias 0 -> 1
- net /RELAY_POWER: track 66.4 -> 62.2 mm
- net +12V: track 243.5 -> 247.4 mm
- net Net-(D1-Pad2): track 9.88 -> 13.5 mm
- net /WIEGAND_D0: track 42.7 -> 39.4 mm
- net /RELAY_CONTACT: track 24.4 -> 27.2 mm
- net +5V: track 217.4 -> 215.2 mm
- net /RELAY_DOOR: track 28.2 -> 29.5 mm
- net /BASE_DOOR_2: track 24.9 -> 24.3 mm
- net /WEMOS_TRIG: track 60.6 -> 61.2 mm
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Other:
- board text added: "Greg J Arnold"
- board text added: "Version 1.1"
